File: GL850G.kicad_sch (KiCad schematic)
At the start: 66 parts, among them J1 Conn_01x03_Pin, J2 5V, J3 5V_OUT, J4 USB_A, J5 USB_A, J9 Conn_01x03_Pin, Q1 40p04, U1 GL850G/GL852G, U11 AP2141WG, U12 USBLC6-2SC6, U2 AP2141WG, U3 AP2141WG, U4 AP2141WG, U5 USBLC6-2SC6, U6 USBLC6-2SC6, Y1 12MHz

Commit message: new file:   0.My_footprint_library.pretty/Standoff_M2.kicad_mod 	new file:   0.My_footprint_library.pretty/USB_2.0_TYPE_A_RECESSED.kicad_mod 	new file:   GL850G-backups/GL850G-2026-01-04_175119.zip 	new file:   GL850G-backups/GL850G-2026-01-04_175654.zip 	new file:   GL850G-backups/GL850G-2026-01-04_180228.zip 	new file:   GL850G-backups/GL850G-2026-01-04_181244.zip 	new file:   GL850G-backups/GL850G-2026-01-04_182825.zip 	modified:   GL850G.kicad_pcb 	modified:   GL850G.kicad_pro 	modified:   GL850G.kicad_sch 	modified:   fp-info-cache 	new file:   fp-lib-table 	modified:   production/GL850G.zip 	deleted:    production/backups/GL850G_2025-12-12_22-37-32.zip 	deleted:    production/backups/GL850G_2026-01-03_19-52-49.zip 	new file:   production/backups/GL850G_2026-01-04_18-14-26.zip 	modified:   production/bom.csv 	modified:   production/designators.csv 	modified:   production/netlist.ipc 	modified:   production/positions.csv 	deleted:    ~GL850G.kicad_pcb.lck
Parts:
- added H1, H2, H3, H4: mount, 0.My_footprint_library:Standoff_M2, symbol Mechanical:MountingHole_Pad
- F1: footprint Capacitor_SMD:C_1812_4532Metric_Pad1.57x3.40mm_HandSolder -> Fuse:Fuseholder_Littelfuse_Nano2_154x
- J4, J5: footprint My_Library:USB_A_2.0 -> 0.My_footprint_library:USB_2.0_TYPE_A_RECESSED
Connections:
- net D0N: now also U12.1 (I/O1); no longer U12.6 (I/O1)
- net D0P: now also U12.3 (I/O2); no longer U12.4 (I/O2)
- net D0_N: now also U12.6 (I/O1); no longer U12.1 (I/O1)
- net D0_P: now also U12.4 (I/O2); no longer U12.3 (I/O2)
- net GND: now also H1.1, H2.1, H3.1, H4.1
Other:
- note added: "- Removed R8 - D9 changed to D2 - Reset jumper removed - D1 fixed polarity - Changed values of R35, R0_2, R10 to adjust LED brightness - Replaced AP2151WG with AP2141WG to fix output logic - Changed electrolytic to ceramic capacitor - Changed USB-A connectors - Added standoff holes - - Added external power supply input - [[ Went back to 0603 components ]]"
- note removed: "- Removed R8 - D9 changed to D2 - Reset jumper removed - D1 fixed polarity - Changed values of R35, R0_2, R10 to adjust LED brightness - Replaced AP2151WG with AP2141WG to fix output logic - Changed electrolytic to ceramic capacitor - [[ Went back to 0603 components ]] - Added external power supply input"
- note removed: "Buy components: 680ohm res"
- note removed: "Find components: BZT52C5V6 B5819W FUSE 2.5A 12pF cap USB 2.0 AP2141WG"
- moved on the sheet: C10, C11, D0_1, J3, R0_1, R0_2, R8, Y1

Commit message: modified:   0.My_footprint_library.pretty/Standoff_M2.kicad_mod 	deleted:    GL850G-backups/GL850G-2025-12-12_214821.zip 	deleted:    GL850G-backups/GL850G-2025-12-12_220756.zip 	deleted:    GL850G-backups/GL850G-2025-12-12_222827.zip 	deleted:    GL850G-backups/GL850G-2025-12-12_223657.zip 	deleted:    GL850G-backups/GL850G-2025-12-12_225255.zip 	deleted:    GL850G-backups/GL850G-2025-12-20_163113.zip 	deleted:    GL850G-backups/GL850G-2025-12-28_152439.zip 	deleted:    GL850G-backups/GL850G-2025-12-29_163703.zip 	new file:   GL850G-backups/GL850G-2026-01-23_173627.zip 	new file:   GL850G-backups/GL850G-2026-01-23_195252.zip 	new file:   GL850G-backups/GL850G-2026-01-23_214158.zip 	new file:   GL850G-backups/GL850G-2026-01-23_220333.zip 	new file:   GL850G-backups/GL850G-2026-01-23_225729.zip 	new file:   GL850G-backups/GL850G-2026-01-24_125535.zip 	new file:   GL850G-backups/GL850G-2026-01-24_131237.zip 	new file:   GL850G-backups/GL850G-2026-01-24_131748.zip 	new file:   GL850G-backups/GL850G-2026-01-24_133206.zip 	new file:   GL850G-backups/GL850G-2026-01-24_133903.zip 	modified:   GL850G.kicad_pcb 	modified:   GL850G.kicad_sch 	new file:   bom/ibom.html 	modified:   fabrication-toolkit-options.json 	modified:   fp-info-cache 	deleted:    production/GL850G.zip 	deleted:    production/backups/GL850G_2026-01-04_18-14-26.zip 	new file:   production/backups/production_V1.2_2026-01-24_13-42-50.zip 	modified:   production/netlist.ipc 	new file:   production/production_V1.2.zip 	renamed:    production/bom.csv -> production/production_V1.2_bom.csv 	renamed:    production/designators.csv -> production/production_V1.2_designators.csv 	renamed:    production/positions.csv -> production/production_V1.2_positions.csv
Parts:
- removed R67, R68: 5.1k_1%, Resistor_SMD:R_0603_1608Metric_Pad0.98x0.95mm_HandSolder, symbol Device:R_Small
- added R11, R12: 5.1k_1%, Resistor_SMD:R_0603_1608Metric_Pad0.98x0.95mm_HandSolder, symbol Device:R_Small
- R1: value 1k -> 5.1k
- R2: value 2k -> 10k
Connections:
- net GND: now also R11.1, R12.1
- net at USB1.A5 (CC1): now also R12.2
- net at USB1.B5 (CC2): now also R11.2
- net 3V renamed pself
Other:
- note added: "- Removed R8 - D9 changed to D2 - Reset jumper removed - Changed values of R35, R0_2, R10 to adjust LED brightness - Replaced AP2151WG with AP2141WG to fix output logic - Changed electrolytic to ceramic capacitor - Changed USB-A connectors - Added standoff holes - Fixed USB uplink traces - Went back to 0603 components"
- note added: "V1.2: Release notes"
- note removed: "- Removed R8 - D9 changed to D2 - Reset jumper removed - D1 fixed polarity - Changed values of R35, R0_2, R10 to adjust LED brightness - Replaced AP2151WG with AP2141WG to fix output logic - Changed electrolytic to ceramic capacitor - Changed USB-A connectors - Added standoff holes - - Added external power supply input - [[ Went back to 0603 components ]]"
- note removed: "V1.0: Release notes"
- title: GL850G_USB_Hub_Reversed -> GL850G_USB_Hub
Changed lines of the file:
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@@
 	(paper "A4")
 	(title_block
-		(title "GL850G_USB_Hub_Reversed")
+		(title "GL850G_USB_Hub")
 		(date "2025-12-08")
 		(rev "1")
 		(company "Stelmach")
-		(comment 1 "Reverse engineered from Aliexpress board")
 	)
 	(rectangle
@@
 		)
 	)
-	(text "V1.0: Release notes"
+	(text "V1.2: Release notes"
 		(exclude_from_sim no)
 		(at 125.73 169.926 0)
@@
 		)
 	)
-	(text "- Removed R8\n- D9 changed to D2\n- Reset jumper removed\n- D1 fixed polarity\n- Changed values of R35, R0_2, R10 to \n   adjust LED brightness\n- Replaced AP2151WG with AP2141WG to fix \n   output logic\n- Changed electrolytic to ceramic capacitor\n- Changed USB-A connectors\n- Added standoff holes\n- \n- Added external power supply input\n- [[ Went back to 0603 components ]]\n"
+	(text "- Removed R8\n- D9 changed to D2\n- Reset jumper removed\n- Changed values of R35, R0_2, R10 to \n   adjust LED brightness\n- Replaced AP2151WG with AP2141WG to fix \n   output logic\n- Changed electrolytic to ceramic capacitor\n- Changed USB-A connectors\n- Added standoff holes\n- Fixed USB uplink traces\n- Went back to 0603 components\n"
 		(exclude_from_sim no)
 		(at 125.73 172.72 0)
@@
 	(wire
 		(pts
-			(xy 252.73 143.51) (xy 264.16 143.51)
+			(xy 252.73 143.51) (xy 265.43 143.51)
 		)
 		(stroke
@@
 	(wire
 		(pts
-			(xy 264.16 142.24) (xy 264.16 143.51)
+			(xy 265.43 142.24) (xy 265.43 143.51)
 		)
 		(stroke
@@
 	)
 	(label "OVCUR_FLG"
-		(at 100.33 144.78 180)
+		(at 100.33 144.78 0)
 		(effects
 			(font
 				(size 1.27 1.27)
 			)
-			(justify right bottom)
+			(justify left bottom)
 		)
 	)
@@
 			)
 		)
-		(property "Value" "2k"
+		(property "Value" "10k"
 			(at 86.614 185.166 0)
 			(effects
@@
 			)
 		)
-		(property "Value" "3V"
+		(property "Value" "pself"
 			(at 114.046 172.974 0)
 			(effects
@@
 		(unit 1)
 		(exclude_from_sim no)
-		(in_bom no)
+		(in_bom yes)
 		(on_board yes)
-		(dnp yes)
-		(property "Reference" "R68"
+		(dnp no)
+		(property "Reference" "R12"
 			(at 53.34 58.674 0)
 			(effects
@@
 			(project "GL850G"
 				(path "/f968fbcd-e4e6-402c-b27d-9750a091b1fe"
-					(reference "R68")
+					(reference "R12")
 					(unit 1)
 				)
@@
 			)
 		)
-		(property "Value" "1k"
+		(property "Value" "5.1k"
 			(at 87.63 179.832 90)
 			(effects
@@
 	)
 	(symbol
+		(lib_id "Device:R_Small")
+		(at 49.53 59.69 180)
+		(unit 1)
+		(exclude_from_sim no)
+		(in_bom yes)
+		(on_board yes)
+		(dnp no)
+		(property "Reference" "R11"
+			(at 48.26 58.674 0)
+			(effects
+				(font
+					(size 1.27 1.27)
+				)
+				(justify left)
+			)
+		)
+		(property "Value" "5.1k_1%"
+			(at 48.26 60.706 0)
+			(effects
+				(font
+					(size 1.27 1.27)
+				)
+				(justify left)
+			)
+		)
+		(property "Footprint" "Resistor_SMD:R_0603_1608Metric_Pad0.98x0.95mm_HandSolder"
+			(at 49.53 59.69 0)
+			(effects
+				(font
+					(size 1.27 1.27)
+				)
+				(hide yes)
+			)
+		)
+		(property "Datasheet" "~"
+			(at 49.53 59.69 0)
+			(effects
+				(font
+					(size 1.27 1.27)
+				)
+				(hide yes)
+			)
+		)
+		(property "Description" "Resistor, small symbol"
+			(at 49.53 59.69 0)
+			(effects
+				(font
+					(size 1.27 1.27)
+				)
+				(hide yes)
+			)
+		)
+		(property "Height" ""
+			(at 49.53 59.69 0)
+			(effects
+				(font
+					(size 1.27 1.27)
+				)
+				(hide yes)
+			)
+		)
+		(property "Manufacturer_Name" ""
+			(at 49.53 59.69 0)
+			(effects
+				(font
+					(size 1.27 1.27)
+				)
+				(hide yes)
+			)
+		)
+		(property "Manufacturer_Part_Number" ""
+			(at 49.53 59.69 0)
+			(effects
+				(font
+					(size 1.27 1.27)
+				)
+				(hide yes)
+			)
+		)
+		(property "Mouser Part Number" ""
+			(at 49.53 59.69 0)
+			(effects
+				(font
+					(size 1.27 1.27)
+				)
+				(hide yes)
+			)
+		)
+		(property "Mouser Price/Stock" ""
+			(at 49.53 59.69 0)
+			(effects
+				(font
+					(size 1.27 1.27)
+				)
+				(hide yes)
+			)
+		)
+		(pin "1"
+		)
+		(pin "2"
+		)
+		(instances
+			(project "GL850G"
+				(path "/f968fbcd-e4e6-402c-b27d-9750a091b1fe"
+					(reference "R11")
+					(unit 1)
+				)
+			)
+		)
+	)
+	(symbol
 		(lib_id "Connector:USB_A")
 		(at 25.4 149.86 0)
@@
 	(symbol
 		(lib_id "power:+3V3")
-		(at 264.16 142.24 0)
+		(at 265.43 142.24 0)
 		(unit 1)
 		(exclude_from_sim no)
@@
 		(dnp no)
 		(property "Reference" "#PWR016"
-			(at 264.16 146.05 0)
+			(at 265.43 146.05 0)
 			(effects
 				(font
@@
 		)
 		(property "Value" "+3V3"
-			(at 263.906 138.684 0)
+			(at 265.176 138.684 0)
 			(effects
 				(font
@@
 		)
 		(property "Footprint" ""
-			(at 264.16 142.24 0)
+			(at 265.43 142.24 0)
 			(effects
 				(font
@@
 		)
 		(property "Datasheet" ""
-			(at 264.16 142.24 0)
+			(at 265.43 142.24 0)
 			(effects
 				(font
@@
 		)
 		(property "Description" "Power symbol creates a global label with name \"+3V3\""
-			(at 264.16 142.24 0)
+			(at 265.43 142.24 0)
 			(effects
 				(font
@@
 			)
 		)
-		(property "Value" "3V"
-			(at 257.81 139.7 90)
+		(property "Value" "pself"
+			(at 258.826 139.446 90)
 			(effects
 				(font
@@
 					(unit 1)
 				)
-			)
-		)
-	)
-	(symbol
-		(lib_id "Device:R_Small")
-		(at 49.53 59.69 180)
-		(unit 1)
-		(exclude_from_sim no)
-		(in_bom no)
-		(on_board yes)
-		(dnp yes)
-		(property "Reference" "R67"
-			(at 48.26 58.674 0)
-			(effects
-				(font
-					(size 1.27 1.27)
-				)
-				(justify left)
-			)
-		)
-		(property "Value" "5.1k_1%"
-			(at 48.26 60.706 0)
-			(effects
-				(font
-					(size 1.27 1.27)
-				)
-				(justify left)
-			)
-		)
-		(property "Footprint" "Resistor_SMD:R_0603_1608Metric_Pad0.98x0.95mm_HandSolder"
-			(at 49.53 59.69 0)
-			(effects
-				(font
-					(size 1.27 1.27)
-				)
-				(hide yes)
-			)
-		)
-		(property "Datasheet" "~"
-			(at 49.53 59.69 0)
-			(effects
-				(font
-					(size 1.27 1.27)
-				)
-				(hide yes)
-			)
-		)
-		(property "Description" "Resistor, small symbol"
-			(at 49.53 59.69 0)
-			(effects
-				(font
-					(size 1.27 1.27)
-				)
-				(hide yes)
-			)
-		)
-		(property "Height" ""
-			(at 49.53 59.69 0)
-			(effects
-				(font
-					(size 1.27 1.27)
-				)
-				(hide yes)
-			)
-		)
-		(property "Manufacturer_Name" ""
-			(at 49.53 59.69 0)
-			(effects
-				(font
-					(size 1.27 1.27)
-				)
-				(hide yes)
-			)
-		)
-		(property "Manufacturer_Part_Number" ""
-			(at 49.53 59.69 0)
-			(effects
-				(font
-					(size 1.27 1.27)
-				)
-				(hide yes)
-			)
-		)
-		(property "Mouser Part Number" ""
-			(at 49.53 59.69 0)
-			(effects
-				(font
-					(size 1.27 1.27)
-				)
-				(hide yes)
-			)
-		)
-		(property "Mouser Price/Stock" ""
-			(at 49.53 59.69 0)
-			(effects
-				(font
-					(size 1.27 1.27)
-				)
-				(hide yes)
-			)
-		)
-		(pin "1"
-		)
-		(pin "2"
-		)
-		(instances
-			(project "GL850G"
-				(path "/f968fbcd-e4e6-402c-b27d-9750a091b1fe"
-					(reference "R67")
-					(unit 1)
-				)
