File: GL850G.kicad_pcb (KiCad board)
At the start: 4 copper layers, 43 parts, among them J1 USB_A, J2 USB_A, J3 USB_A, J4 USB_A, J5 USB_A, U1 GL850G, Y1 12MHz

Commit message: Add files via upload
Parts:
- removed C3, C4: ?, Capacitor_SMD:C_0805_2012Metric_Pad1.18x1.45mm_HandSolder
- added C14: 2.2uF, Capacitor_SMD:C_0603_1608Metric_Pad1.08x0.95mm_HandSolder, F.Cu at (162.6, 87.5)
- added C15: 2.2uF, Capacitor_SMD:C_0603_1608Metric_Pad1.08x0.95mm_HandSolder, F.Cu at (162.7, 94.5)
- added D9: LED, LED_SMD:LED_0805_2012Metric_Pad1.15x1.40mm_HandSolder, F.Cu at (164.1, 82.0)
- added J6: Conn_01x03_Pin, Connector_PinHeader_2.54mm:PinHeader_1x03_P2.54mm_Vertical, F.Cu at (169.1, 99.4)
- added J7: Conn_01x02_Pin, Connector_PinHeader_2.54mm:PinHeader_1x02_P2.54mm_Vertical, F.Cu at (120.2, 102.1)
- added J8: Conn_01x02_Pin, Connector_PinHeader_2.54mm:PinHeader_1x02_P2.54mm_Vertical, F.Cu at (155.4, 110.5)
- added J9: Conn_01x03_Pin, Connector_PinHeader_2.54mm:PinHeader_1x03_P2.54mm_Vertical, F.Cu at (169.4, 115.8)
- added R35: 330, Resistor_SMD:R_0805_2012Metric_Pad1.20x1.40mm_HandSolder, F.Cu at (169.0, 82.0)
- added U11: AP2151WG, Package_TO_SOT_SMD:SOT-23-5_HandSoldering, F.Cu at (162.7, 91.0)
- moved J2 148.6 mm to (177.0, 92.0), turned to 90 degrees
- moved C8 147.8 mm to (173.2, 113.4), turned to -90 degrees
- moved J5 142.0 mm to (177.0, 108.4), turned to 90 degrees
- moved C5 139.5 mm to (173.3, 97.0), turned to -90 degrees
- moved J1 120.3 mm to (146.8, 76.3), turned to 180 degrees
- moved R1 120.1 mm to (157.0, 95.1), turned to 90 degrees
- moved C9 115.4 mm to (147.8, 96.1), turned to -90 degrees
- moved J4 113.2 mm to (143.9, 111.0)
- moved F1 113.2 mm to (158.4, 75.8)
- moved R8 112.7 mm to (150.1, 96.1), turned to -90 degrees
- moved C7 112.7 mm to (139.9, 107.9)
- moved C1 111.1 mm to (157.3, 81.3), turned to -90 degrees
- moved TP5 110.2 mm to (159.9, 97.6)
- moved TP4 109.6 mm to (158.2, 89.6), turned to 180 degrees
- moved R0_2 108.0 mm to (154.4, 96.1), turned to 90 degrees
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Connections:
- C5 pad 1: +5V -> Net-(J2-VBUS)
- C6 pad 1: +5V -> Net-(J3-VBUS)
- C7 pad 1: +5V -> Net-(J4-VBUS)
- C8 pad 1: +5V -> Net-(J5-VBUS)
- J2 pad 1: +5V -> Net-(J2-VBUS)
- J3 pad 1: +5V -> Net-(J3-VBUS)
- J4 pad 1: +5V -> Net-(J4-VBUS)
- J5 pad 1: +5V -> Net-(J5-VBUS)
- TP2 pad 1: unconnected-(TP2-Pad1) -> /D2P
- TP3 pad 1: unconnected-(TP3-Pad1) -> /D2M
Other:
- board outline added: 75 x 60 mm

Commit message: Add files via upload
Parts:
- removed TP2, TP3: TestPoint, TestPoint:TestPoint_Pad_D2.0mm
- moved R2 78.4 mm to (215.8, 76.7)
- moved R1 65.2 mm to (220.8, 81.8)
- moved C9 57.1 mm to (198.2, 69.3)
- moved D1 57.1 mm to (196.8, 64.2)
- moved R8 57.1 mm to (200.6, 69.4)
- moved R10 57.1 mm to (199.9, 65.2)
- moved R5 57.1 mm to (196.1, 69.4)
- moved R6 57.1 mm to (196.8, 66.3)
- moved C1 44.4 mm to (200.2, 92.9), turned to 0 degrees
- moved TP7 37.2 mm to (105.0, 101.1)
- moved TP6 37.2 mm to (105.1, 104.2)
- moved R7 30.9 mm to (106.1, 81.6)
- moved C8 20.3 mm to (155.7, 103.1), turned to 180 degrees
- moved R35 19.7 mm to (170.6, 101.7), turned to 180 degrees
- moved R0_2 18.3 mm to (168.5, 84.3), turned to 0 degrees
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Connections:
- net /D0M renamed /D0N
- net /D1M renamed /D1N
- net /D3M renamed /D3N
- J3 pad 2: /D2M -> /D4N
- J3 pad 3: /D2P -> /D4P
- J5 pad 2: /D4M -> /D2N
- J5 pad 3: /D4P -> /D2P
- U1 pad 11: /D4M -> /D4N
- U1 pad 2: /D2M -> /D2N
Routing:
- net /D2P: track 0.00 -> 54.2 mm
- net /D2N: track 0.00 -> 53.6 mm
- net /D4N: track 0.00 -> 42.1 mm
- net /D4P: track 0.00 -> 40.3 mm
- net /D3N: track 0.00 -> 39.4 mm, vias 0 -> 1
- net /D3P: track 0.00 -> 37.6 mm, vias 0 -> 1
- net /D1N: track 0.00 -> 26.3 mm, vias 0 -> 2
- net /D1P: track 0.00 -> 26.1 mm, vias 0 -> 2
- net /D0N: track 0.00 -> 17.7 mm
- net /D0P: track 0.00 -> 17.1 mm
- net /HSE_in: track 0.00 -> 11.6 mm
- net /HSE_out: track 0.00 -> 10.1 mm
Other:
- board size 75 x 60 mm -> 75 x 55 mm
- board text added: "Stackup: JLC0416H-3313"

Commit message: Add files via upload
Parts:
- added J10: Conn_01x02_Pin, Connector_PinHeader_2.54mm:PinHeader_1x02_P2.54mm_Vertical, F.Cu at (198.3, 66.6)
- added TP2: TestPoint, TestPoint:TestPoint_Pad_D2.0mm, F.Cu at (170.2, 95.6)
- added TP3: TestPoint, TestPoint:TestPoint_Pad_D2.0mm, F.Cu at (198.6, 76.7)
- moved C9 54.5 mm to (149.9, 94.5)
- moved R8 54.5 mm to (152.2, 94.5)
- moved R5 54.5 mm to (147.7, 94.4)
- moved TP6 48.9 mm to (151.7, 89.7)
- moved D0_1 45.6 mm to (213.9, 86.2)
- moved R0_2 45.6 mm to (214.0, 82.4)
- moved TP7 43.5 mm to (147.1, 90.0)
- moved C1 35.1 mm to (169.7, 75.5), turned to -90 degrees
- moved TP1 28.1 mm to (131.4, 101.9)
- moved D9 25.5 mm to (196.1, 98.0)
- moved R35 25.5 mm to (196.1, 100.7)
- moved R7 23.0 mm to (123.6, 96.6)
- moved TP8 21.2 mm to (127.5, 95.6)
- moved R2 21.1 mm to (198.6, 88.8)
- moved R1 21.1 mm to (203.6, 93.9)
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Connections:
- C12 pad 1: Net-(U1-RST) -> /RST
- R7 pad 2: Net-(U1-RST) -> Net-(J10-Pin_2)
- TP8 pad 1: Net-(U1-RST) -> /RST
- U1 pad 13: Net-(U1-RST) -> /RST
Routing:
- net /D1P: track 26.1 -> 106.0 mm, vias 2 -> 0
- net /D1N: track 26.3 -> 105.4 mm, vias 2 -> 0
- net GND: track 0.00 -> 43.7 mm
- net +3V3: track 0.00 -> 29.3 mm
- net /PWREN1: track 0.00 -> 28.9 mm
- net VBUS_out: track 0.00 -> 28.6 mm
- net /OVCUR1: track 0.00 -> 26.4 mm
- net Net-(C2-Pad2): track 0.00 -> 18.1 mm, vias 0 -> 3
- net +5V: track 0.00 -> 16.6 mm
- net (no net): track 0.00 -> 15.0 mm
- net 3V: track 0.00 -> 13.1 mm
- net /PWREN2: track 0.00 -> 11.5 mm
- net Net-(J5-VBUS): track 0.00 -> 10.2 mm
- net Net-(U1-V5): track 0.00 -> 7.97 mm
- net Net-(J2-VBUS): track 0.00 -> 7.73 mm
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Other:
- board text added: "Dsgn date: 2025-12-11"
- board text added: "git:@TheStelmach"

Commit message: Add files via upload
Parts:
- added R11: 100k, Resistor_SMD:R_0805_2012Metric_Pad1.20x1.40mm_HandSolder, F.Cu at (119.4, 84.9)
- moved J10 82.4 mm to (119.4, 90.4)
- moved D0_1 44.0 mm to (170.1, 90.4)
- moved R0_2 40.0 mm to (174.7, 90.4), turned to 180 degrees
- moved R6 29.7 mm to (170.1, 85.6)
- moved D1 29.6 mm to (170.1, 83.5)
- moved R10 29.3 mm to (173.6, 84.5)
- moved R1 25.4 mm to (179.2, 86.9), turned to 0 degrees
- moved TP3 24.8 mm to (174.0, 79.2)
- moved D9 21.7 mm to (174.6, 94.7)
- moved R2 20.4 mm to (179.2, 82.6), turned to 180 degrees
- moved R35 18.0 mm to (179.5, 93.7), turned to 90 degrees
Routing:
- net +5V: track 16.6 -> 252.0 mm, vias 0 -> 4
- net GND: track 43.7 -> 91.8 mm, vias 0 -> 65
- net +3V3: track 29.3 -> 68.6 mm, vias 0 -> 2
- net /PGANG/SUSP: track 4.00 -> 39.7 mm, vias 1 -> 2
- net /RST: track 0.00 -> 25.9 mm
- net /OVCUR1: track 26.4 -> 49.8 mm
- net (no net): track 15.0 -> 0.00 mm
- net Net-(U1-TEST/SCL): track 2.29 -> 12.9 mm
- net /PWREN1: track 28.9 -> 34.9 mm
- net Net-(J10-Pin_2): track 0.00 -> 5.30 mm
- net Net-(D9-K): track 0.00 -> 3.88 mm
- net VBUS_out: track 28.6 -> 32.3 mm
- net Net-(D0_1-A): track 0.00 -> 2.74 mm
- net Net-(D1-K): track 0.00 -> 2.40 mm
- net /D1N: track 105.4 -> 103.1 mm
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- added copper zone on B.Cu, net GND
- added copper zone on In1.Cu, net GND
- added copper zone on In2.Cu, net GND
Other:
- board text added: "Dsgn date: 2025-12-12"
- board text added: "GL850G/GL852G USB Hub Testing board"
- board text added: "OVCUR1"
- board text added: "OVCUR2"
- board text added: "PGANG/SUSP"
- board text added: "PWREN1"
- board text added: "PWREN2"
- board text added: "RST"
- board text added: "TEST"
- board text added: "VBUS_out"
- board text removed: "Dsgn date: 2025-12-11"

Commit message: deleted:    GL850G-backups/GL850G-2025-12-08_201710.zip 	deleted:    GL850G-backups/GL850G-2025-12-08_202241.zip 	deleted:    GL850G-backups/GL850G-2025-12-08_202819.zip 	deleted:    GL850G-backups/GL850G-2025-12-08_203416.zip 	deleted:    GL850G-backups/GL850G-2025-12-08_204521.zip 	deleted:    GL850G-backups/GL850G-2025-12-09_212715.zip 	deleted:    GL850G-backups/GL850G-2025-12-09_213849.zip 	deleted:    GL850G-backups/GL850G-2025-12-09_214411.zip 	deleted:    GL850G-backups/GL850G-2025-12-09_215034.zip 	deleted:    GL850G-backups/GL850G-2025-12-09_215627.zip 	deleted:    GL850G-backups/GL850G-2025-12-10_200556.zip 	deleted:    GL850G-backups/GL850G-2025-12-10_201346.zip 	deleted:    GL850G-backups/GL850G-2025-12-10_202529.zip 	deleted:    GL850G-backups/GL850G-2025-12-10_203150.zip 	deleted:    GL850G-backups/GL850G-2025-12-10_203933.zip 	deleted:    GL850G-backups/GL850G-2025-12-11_155218.zip 	deleted:    GL850G-backups/GL850G-2025-12-11_155719.zip 	deleted:    GL850G-backups/GL850G-2025-12-11_160353.zip 	deleted:    GL850G-backups/GL850G-2025-12-11_160919.zip 	deleted:    GL850G-backups/GL850G-2025-12-11_161458.zip 	new file:   GL850G-backups/GL850G-2025-12-12_214821.zip 	new file:   GL850G-backups/GL850G-2025-12-12_220756.zip 	new file:   GL850G-backups/GL850G-2025-12-12_222827.zip 	new file:   GL850G-backups/GL850G-2025-12-12_223657.zip 	new file:   GL850G-backups/GL850G-2025-12-12_225255.zip 	new file:   GL850G-backups/GL850G-2025-12-20_163113.zip 	new file:   GL850G-backups/GL850G-2025-12-28_152439.zip 	new file:   GL850G-backups/GL850G-2025-12-29_163703.zip 	new file:   GL850G-backups/GL850G-2025-12-29_182820.zip 	modified:   GL850G.kicad_pcb 	modified:   GL850G.kicad_prl 	modified:   GL850G.kicad_pro 	modified:   GL850G.kicad_sch 	new file:   GL850G.png 	new file:   GL850G_back.png 	new file:   fabrication-toolkit-options.json 	modified:   fp-info-cache 	new file:   production/GL850G.zip 	new file:   production/backups/GL850G_2025-12-12_22-37-32.zip 	new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
Parts:
- C13, C5, C6, C7, C8, C9: footprint Capacitor_SMD:C_0805_2012Metric_Pad1.18x1.45mm_HandSolder -> Capacitor_SMD:C_0603_1608Metric_Pad1.08x0.95mm_HandSolder
- C2: value ? -> 100nF; footprint Capacitor_SMD:C_0805_2012Metric_Pad1.18x1.45mm_HandSolder -> Capacitor_SMD:C_0603_1608Metric_Pad1.08x0.95mm_HandSolder
- R35: value 330 -> 500
- moved C8 0.21 mm to (154.4, 103.1)
- moved C2 0.20 mm to (133.5, 77.9)
- moved C9 0.16 mm to (149.9, 94.3)
- moved C7 0.16 mm to (137.3, 103.1)
- moved C13 0.16 mm to (142.0, 79.8)
- moved C6 0.11 mm to (120.5, 103.1)
- moved C5 0.05 mm to (173.0, 102.9), turned to 0 degrees
Routing:
- net Net-(J3-VBUS): track 6.87 -> 7.43 mm
- net GND: track 91.8 -> 91.5 mm, vias 65 -> 73
- added copper zone on F.Cu, net GND

Commit message: modified:   0.My_Library.bak 	modified:   0.My_Library.kicad_sym 	new file:   GL850G-backups/GL850G-2026-01-02_150657.zip 	new file:   GL850G-backups/GL850G-2026-01-02_151627.zip 	new file:   GL850G-backups/GL850G-2026-01-02_160446.zip 	new file:   GL850G-backups/GL850G-2026-01-03_192335.zip 	new file:   GL850G-backups/GL850G-2026-01-03_193700.zip 	new file:   GL850G-backups/GL850G-2026-01-03_194723.zip 	new file:   GL850G-backups/GL850G-2026-01-03_195234.zip 	new file:   GL850G-backups/GL850G-2026-01-03_195824.zip 	modified:   GL850G.kicad_pcb 	modified:   GL850G.kicad_pro 	modified:   GL850G.kicad_sch 	new file:   GL850G_USB_Hub_BACKUP.zip 	modified:   fp-info-cache 	modified:   production/GL850G.zip 	new file:   production/backups/GL850G_2026-01-03_19-52-49.zip 	modified:   production/bom.csv 	modified:   production/designators.csv 	modified:   production/netlist.ipc 	modified:   production/positions.csv
Parts:
- removed D9: LED, LED_SMD:LED_0805_2012Metric_Pad1.15x1.40mm_HandSolder
- removed J10, J7, J8: Conn_01x02_Pin, Connector_PinHeader_2.54mm:PinHeader_1x02_P2.54mm_Vertical
- removed J6: Conn_01x03_Pin, Connector_PinHeader_2.54mm:PinHeader_1x03_P2.54mm_Vertical
- removed R11: 100k, Resistor_SMD:R_0805_2012Metric_Pad1.20x1.40mm_HandSolder
- removed R35: 500, Resistor_SMD:R_0805_2012Metric_Pad1.20x1.40mm_HandSolder
- removed TP1, TP3, TP4, TP6, TP7, TP8: TestPoint, TestPoint:TestPoint_Pad_D2.0mm
- added C16: 2.2uF, Capacitor_SMD:C_0603_1608Metric_Pad1.08x0.95mm_HandSolder, F.Cu at (140.8, 91.8)
- added C17: 2.2uF, Capacitor_SMD:C_0603_1608Metric_Pad1.08x0.95mm_HandSolder, F.Cu at (134.1, 91.8)
- added C18: 2.2uF, Capacitor_SMD:C_0603_1608Metric_Pad1.08x0.95mm_HandSolder, F.Cu at (131.3, 93.1)
- added C19: 2.2uF, Capacitor_SMD:C_0603_1608Metric_Pad1.08x0.95mm_HandSolder, F.Cu at (124.7, 93.1)
- added C3: 2.2uF, Capacitor_SMD:C_0603_1608Metric_Pad1.08x0.95mm_HandSolder, F.Cu at (152.9, 91.8)
- added C4: 2.2uF, Capacitor_SMD:C_0603_1608Metric_Pad1.08x0.95mm_HandSolder, F.Cu at (146.2, 91.9)
- added D2: LED, LED_SMD:LED_0805_2012Metric_Pad1.15x1.40mm_HandSolder, F.Cu at (144.1, 76.0)
- added D7: BZT52C5V6, Diode_SMD:D_SOD-123, F.Cu at (174.8, 85.4)
- added D8: B5819W, Diode_SMD:D_SOD-123, F.Cu at (174.8, 88.1)
- added F4: 500mA, Fuse:Fuse_0805_2012Metric, F.Cu at (153.8, 70.2)
- added Q1: 40p04, Package_TO_SOT_SMD:TO-252-2, F.Cu at (168.1, 74.6)
- added R13: 5.1k_1%, Resistor_SMD:R_0603_1608Metric_Pad0.98x0.95mm_HandSolder, B.Cu at (172.3, 109.8)
- added R14: 5.1k_1%, Resistor_SMD:R_0603_1608Metric_Pad0.98x0.95mm_HandSolder, B.Cu at (169.8, 109.8)
- added R15: 5.1k_1%, Resistor_SMD:R_0603_1608Metric_Pad0.98x0.95mm_HandSolder, B.Cu at (123.8, 109.7)
- added R16: 5.1k_1%, Resistor_SMD:R_0603_1608Metric_Pad0.98x0.95mm_HandSolder, B.Cu at (121.3, 109.7)
- added R26: 10k, Resistor_SMD:R_0603_1608Metric_Pad0.98x0.95mm_HandSolder, F.Cu at (175.0, 67.5)
- added R67: 5.1k_1%, Resistor_SMD:R_0603_1608Metric_Pad0.98x0.95mm_HandSolder, B.Cu at (145.3, 67.5)
- added R68: 5.1k_1%, Resistor_SMD:R_0603_1608Metric_Pad0.98x0.95mm_HandSolder, B.Cu at (148.1, 67.5)
- added U12: USBLC6-2SC6, Package_TO_SOT_SMD:SOT-23-6, F.Cu at (134.6, 70.6)
- added U2: AP2141WG, Package_TO_SOT_SMD:SOT-23-5_HandSoldering, F.Cu at (149.6, 91.9)
- added U3: AP2141WG, Package_TO_SOT_SMD:SOT-23-5_HandSoldering, F.Cu at (137.4, 91.8)
- added U4: AP2141WG, Package_TO_SOT_SMD:SOT-23-5_HandSoldering, F.Cu at (128.0, 93.1)
- added U5: USBLC6-2SC6, Package_TO_SOT_SMD:SOT-23-6, F.Cu at (171.6, 101.1)
- added U6: USBLC6-2SC6, Package_TO_SOT_SMD:SOT-23-6, F.Cu at (122.4, 100.7)
- added USB1: USB_C_Recep._USB2.0_16P, Connector_USB:USB_C_Receptacle_GCT_USB4105-xx-A_16P_TopMnt_Horizontal, F.Cu at (146.8, 67.0)
- added USB2: USB_C_Recep._USB2.0_16P, Connector_USB:USB_C_Receptacle_GCT_USB4105-xx-A_16P_TopMnt_Horizontal, F.Cu at (171.1, 110.0)
- added USB3: USB_C_Recep._USB2.0_16P, Connector_USB:USB_C_Receptacle_GCT_USB4105-xx-A_16P_TopMnt_Horizontal, F.Cu at (122.5, 110.0)
- C1: footprint Capacitor_THT:CP_Radial_D5.0mm_P2.00mm -> Capacitor_SMD:C_1206_3216Metric_Pad1.33x1.80mm_HandSolder
- C5, C6: value 100nF -> 100uF; footprint Capacitor_SMD:C_0603_1608Metric_Pad1.08x0.95mm_HandSolder -> Capacitor_SMD:C_1206_3216Metric_Pad1.33x1.80mm_HandSolder
- F1: value Fuse_Small -> Fuse; footprint Fuse:Fuse_1210_3225Metric_Pad1.42x2.65mm_HandSolder -> Capacitor_SMD:C_1812_4532Metric_Pad1.57x3.40mm_HandSolder
- J1: value USB_A -> Conn_01x03_Pin; footprint My_Library:USB_A_2.0 -> Connector_PinHeader_2.54mm:PinHeader_1x03_P2.54mm_Vertical
- J2: value USB_A -> 5V; footprint My_Library:USB_A_2.0 -> Connector_JST:JST_XH_B2B-XH-A_1x02_P2.50mm_Vertical
- J3: value USB_A -> 5V_OUT; footprint My_Library:USB_A_2.0 -> Connector_PinHeader_2.54mm:PinHeader_1x02_P2.54mm_Vertical
- R0_2: value 100k -> 1k
- R1: value 10k -> 1k
- R10: value 1k -> 2k
- R2: value 20k -> 2k
- R8: value ? -> 1k; footprint Capacitor_SMD:C_0805_2012Metric_Pad1.18x1.45mm_HandSolder -> Resistor_SMD:R_0805_2012Metric_Pad1.20x1.40mm_HandSolder
- U1: value GL850G -> GL850G/GL852G
- U11: value AP2151WG -> AP2141WG
- moved C6 59.1 mm to (174.9, 80.0)
- moved R0_2 56.5 mm to (122.1, 70.0)
- moved J3 51.3 mm to (176.4, 97.1)
- moved D0_1 48.1 mm to (126.6, 70.0)
- moved R1 41.6 mm to (139.0, 76.0), turned to -90 degrees
- moved J2 41.1 mm to (166.9, 66.1)
- moved R2 38.2 mm to (141.5, 76.1), turned to 90 degrees
- moved R10 27.4 mm to (146.2, 83.2), turned to 90 degrees
- moved J1 26.7 mm to (134.6, 95.7), turned to 90 degrees
- moved D1 26.4 mm to (143.7, 83.2), turned to 90 degrees
- moved R6 21.6 mm to (148.7, 83.2), turned to 90 degrees
- moved C5 20.2 mm to (174.9, 82.7), turned to 180 degrees
- moved R8 19.3 mm to (146.5, 76.1), turned to 90 degrees
- moved C1 17.0 mm to (155.2, 66.6), turned to 180 degrees
- moved C15 12.9 mm to (168.3, 94.8), turned to 90 degrees
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Connections:
- C15 pad 1: VBUS_out -> VBUS_out1
- C5 pad 1: Net-(J2-VBUS) -> Net-(D7-K)
- C6 pad 1: Net-(J3-VBUS) -> Net-(D7-K)
- C7 pad 1: Net-(J4-VBUS) -> Net-(J1-Pin_2)
- D0_1 pad 1: /PWREN1 -> Net-(D0_1-K)
- D0_1 pad 2: Net-(D0_1-A) -> +3V3
- D1 pad 1: Net-(D1-K) -> /PGANG/SUSP
- D1 pad 2: /PGANG/SUSP -> Net-(D1-A)
- F1 pad 1: Net-(J1-VBUS) -> Net-(D8-K)
- J1 pad 1: Net-(J1-VBUS) -> +5V
- J1 pad 2: /D0N -> Net-(J1-Pin_2)
- J1 pad 3: /D0P -> VBUS_out3
- J2 pad 1: Net-(J2-VBUS) -> Net-(J2-Pin_1)
- J2 pad 2: /D1N -> GND
- J3 pad 1: Net-(J3-VBUS) -> +5V
- J3 pad 2: /D4N -> GND
- J4 pad 1: Net-(J4-VBUS) -> Net-(J1-Pin_2)
- J9 pad 3: VBUS_out -> VBUS_out2
- R0_2 pad 1: +3V3 -> Net-(D0_1-K)
- R0_2 pad 2: Net-(D0_1-A) -> GND
- R1 pad 1: /OVCUR1 -> Net-(D2-A)
- R10 pad 1: Net-(D1-K) -> +3V3
- R10 pad 2: +3V3 -> Net-(D1-A)
- R2 pad 2: /OVCUR1 -> Net-(D2-A)
- R7 pad 2: Net-(J10-Pin_2) -> /RST
- R8 pad 1: 3V -> /OVCUR1
- R8 pad 2: GND -> Net-(D2-A)
- TP2 pad 1: VBUS_out -> /PWREN1
- U1 pad 14: Net-(U1-TEST/SCL) -> GND
- U1 pad 19: /OVCUR2 -> unconnected-(U1-OVCUR2-Pad19)
- U1 pad 20: /PWREN2 -> unconnected-(U1-PWREN2-Pad20)
- U11 pad 1: VBUS_out -> VBUS_out1
- U11 pad 3: /OVCUR1 -> /OVCUR_FLG
Routing:
- net +5V: track 252.0 -> 23.7 mm, vias 4 -> 17
- net /OVCUR_FLG: track 0.00 -> 113.6 mm, vias 0 -> 5
- net /PWREN1: track 34.9 -> 121.1 mm, vias 0 -> 3
- net /D1N: track 103.1 -> 54.7 mm, vias 0 -> 2
- net /D1P: track 103.7 -> 55.3 mm, vias 0 -> 2
- net VBUS_out: track 32.3 -> 0.00 mm
- net VBUS_out4: track 0.00 -> 24.9 mm
- net /PGANG/SUSP: track 39.7 -> 17.1 mm
- net VBUS_out1: track 0.00 -> 21.9 mm
- net /D4N: track 39.4 -> 18.6 mm
- net +3V3: track 68.6 -> 48.2 mm
- net /D4P: track 37.6 -> 18.0 mm
- net Net-(D7-K): track 0.00 -> 18.2 mm
- net /D0_P: track 0.00 -> 14.8 mm
- net /RST: track 25.9 -> 11.3 mm, vias 0 -> 2
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- added copper zone on B.Cu, net +5V
- added copper zone on F.Cu, net +5V
- removed copper zone on B.Cu, net GND
- removed copper zone on F.Cu, net GND
Other:
- board size 75 x 55 mm -> 65 x 50 mm
- board text added: "Dsgn date: 2026-01-03"
- board text added: "EXT PWR 5V"
- board text added: "GL850G/GL852G USB Hub V1.1"
- board text added: "PORT 1"
- board text added: "PORT 2"
- board text added: "PORT 3"
- board text added: "PORT 4"
- board text added: "PWR"
- board text removed: "Dsgn date: 2025-12-12"
- board text removed: "GL850G/GL852G USB Hub Testing board"
- board text removed: "OVCUR1"
- board text removed: "OVCUR2"
- board text removed: "PGANG/SUSP"
- board text removed: "PWREN1"
- board text removed: "PWREN2"
- board text removed: "RST"
- board text removed: "TEST"
- board text removed: "VBUS_out"

Commit message: new file:   0.My_footprint_library.pretty/Standoff_M2.kicad_mod 	new file:   0.My_footprint_library.pretty/USB_2.0_TYPE_A_RECESSED.kicad_mod 	new file:   GL850G-backups/GL850G-2026-01-04_175119.zip 	new file:   GL850G-backups/GL850G-2026-01-04_175654.zip 	new file:   GL850G-backups/GL850G-2026-01-04_180228.zip 	new file:   GL850G-backups/GL850G-2026-01-04_181244.zip 	new file:   GL850G-backups/GL850G-2026-01-04_182825.zip 	modified:   GL850G.kicad_pcb 	modified:   GL850G.kicad_pro 	modified:   GL850G.kicad_sch 	modified:   fp-info-cache 	new file:   fp-lib-table 	modified:   production/GL850G.zip 	deleted:    production/backups/GL850G_2025-12-12_22-37-32.zip 	deleted:    production/backups/GL850G_2026-01-03_19-52-49.zip 	new file:   production/backups/GL850G_2026-01-04_18-14-26.zip 	modified:   production/bom.csv 	modified:   production/designators.csv 	modified:   production/netlist.ipc 	modified:   production/positions.csv 	deleted:    ~GL850G.kicad_pcb.lck
Parts:
- added H1: mount, 0.My_footprint_library:Standoff_M2, F.Cu at (117.3, 66.5)
- added H2: mount, 0.My_footprint_library:Standoff_M2, F.Cu at (176.3, 66.5)
- added H3: mount, 0.My_footprint_library:Standoff_M2, F.Cu at (117.3, 95.0)
- added H4: mount, 0.My_footprint_library:Standoff_M2, F.Cu at (176.3, 95.0)
- F1: footprint Capacitor_SMD:C_1812_4532Metric_Pad1.57x3.40mm_HandSolder -> Fuse:Fuseholder_Littelfuse_Nano2_154x
- J4, J5: footprint My_Library:USB_A_2.0 -> 0.My_footprint_library:USB_2.0_TYPE_A_RECESSED
- moved J3 2.74 mm to (176.3, 99.8)
- moved R26 2.40 mm to (172.6, 67.4)
- moved C16 1.76 mm to (140.0, 93.4)
- moved C17 1.76 mm to (133.3, 93.4)
- moved J1 1.76 mm to (133.8, 97.3)
- moved U3 1.76 mm to (136.7, 93.4)
- moved C7 1.63 mm to (131.0, 98.7)
- moved J4 1.50 mm to (137.5, 102.5)
- moved J5 1.50 mm to (156.1, 102.5)
- moved C3 1.41 mm to (153.7, 93.0)
- moved C4 1.41 mm to (147.0, 93.0)
- moved J9 1.41 mm to (157.7, 97.0)
- moved U2 1.41 mm to (150.3, 93.1)
- moved C8 1.41 mm to (149.5, 97.7)
- moved F1 1.15 mm to (168.7, 84.2)
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Connections:
- U12 pad 1: /D0_N -> /D0N
- U12 pad 3: /D0_P -> /D0P
- U12 pad 4: /D0P -> /D0_P
- U12 pad 6: /D0N -> /D0_N
Routing:
- net +5V: track 23.7 -> 44.9 mm, vias 17 -> 24
- net /OVCUR_FLG: track 113.6 -> 96.8 mm, vias 5 -> 4
- net /PWREN1: track 121.1 -> 106.4 mm, vias 3 -> 0
- net /D2P: track 57.7 -> 51.3 mm, vias 1 -> 2
- net /D2N: track 57.1 -> 51.9 mm, vias 1 -> 2
- net GND: track 82.6 -> 80.2 mm, vias 37 -> 56
- net /D3N: track 43.2 -> 41.7 mm, vias 0 -> 1
- net Net-(Q1-G): track 12.7 -> 11.6 mm
- net /D3P: track 41.4 -> 40.5 mm, vias 0 -> 1
- net Net-(D7-K): track 18.2 -> 19.1 mm
- net /D0_P: track 14.8 -> 14.1 mm
- net /D0_N: track 14.2 -> 14.7 mm
Other:
- outline, holes or cut-outs redrawn
- board text added: "Dsgn date: 2026-01-04"
- board text removed: "Dsgn date: 2026-01-03"

Commit message: modified:   0.My_footprint_library.pretty/Standoff_M2.kicad_mod 	deleted:    GL850G-backups/GL850G-2025-12-12_214821.zip 	deleted:    GL850G-backups/GL850G-2025-12-12_220756.zip 	deleted:    GL850G-backups/GL850G-2025-12-12_222827.zip 	deleted:    GL850G-backups/GL850G-2025-12-12_223657.zip 	deleted:    GL850G-backups/GL850G-2025-12-12_225255.zip 	deleted:    GL850G-backups/GL850G-2025-12-20_163113.zip 	deleted:    GL850G-backups/GL850G-2025-12-28_152439.zip 	deleted:    GL850G-backups/GL850G-2025-12-29_163703.zip 	new file:   GL850G-backups/GL850G-2026-01-23_173627.zip 	new file:   GL850G-backups/GL850G-2026-01-23_195252.zip 	new file:   GL850G-backups/GL850G-2026-01-23_214158.zip 	new file:   GL850G-backups/GL850G-2026-01-23_220333.zip 	new file:   GL850G-backups/GL850G-2026-01-23_225729.zip 	new file:   GL850G-backups/GL850G-2026-01-24_125535.zip 	new file:   GL850G-backups/GL850G-2026-01-24_131237.zip 	new file:   GL850G-backups/GL850G-2026-01-24_131748.zip 	new file:   GL850G-backups/GL850G-2026-01-24_133206.zip 	new file:   GL850G-backups/GL850G-2026-01-24_133903.zip 	modified:   GL850G.kicad_pcb 	modified:   GL850G.kicad_sch 	new file:   bom/ibom.html 	modified:   fabrication-toolkit-options.json 	modified:   fp-info-cache 	deleted:    production/GL850G.zip 	deleted:    production/backups/GL850G_2026-01-04_18-14-26.zip 	new file:   production/backups/production_V1.2_2026-01-24_13-42-50.zip 	modified:   production/netlist.ipc 	new file:   production/production_V1.2.zip 	renamed:    production/bom.csv -> production/production_V1.2_bom.csv 	renamed:    production/designators.csv -> production/production_V1.2_designators.csv 	renamed:    production/positions.csv -> production/production_V1.2_positions.csv
Parts:
- H1, H2, H3, H4: moved to B.Cu
- R1: value 1k -> 5.1k
- R2: value 2k -> 10k
- turned H1 to 180 degrees
- turned H2 to 180 degrees
- turned H3 to 180 degrees
- turned H4 to 180 degrees
- renumbered R67 to R11, R68 to R12
Connections:
- net 3V renamed pself
Routing:
- net Net-(F4-Pad1): track 14.2 -> 17.1 mm
- net /D4_N: track 4.96 -> 7.48 mm
- net /D1_P: track 4.42 -> 6.84 mm
- net /D0_P: track 14.1 -> 15.9 mm
- net /D4_P: track 4.96 -> 6.67 mm
- net /D1_N: track 4.42 -> 6.12 mm
- net /D0_N: track 14.7 -> 15.7 mm
- net GND: vias 56 -> 72
- net +5V: vias 24 -> 27
Other:
- board text added: "Dsgn date: 2026-01-24"
- board text added: "GL850G/GL852G USB Hub V1.2"
- board text added: "May the board enumerate on the first try and your dmesg be error-free!"
- board text added: "Please enumerate this time, you temperamental silicon diva."
- board text added: "X"
- board text removed: "Dsgn date: 2026-01-04"
- board text removed: "GL850G/GL852G USB Hub V1.1"
